File: magsafe-trigger.kicad_pcb (KiCad board)
At the start: 2 copper layers, 40.2 x 21.5 mm, 12 parts, among them J1 MagSafe 2 female, J2 ID_LED, J3 2.54mm Output, J4 VCC, J5 GND, Q1 IRF3708

Commit message: Update PCB connect MOSFET tab to output gnd
- Add more labels
- Remove back exposed copper
Connections:
- net Net-(D1-Pad2) renamed /GATE
Other:
- board text added: "10V Zener"
- board text added: "MagSafe 2 Trigger github.com/jonathonlui/magsafe-trigger"
- board text added: "OUTPUT"
