File: magsafe-trigger.sch (KiCad schematic (older format))
At the start: 11 parts, among them J1 MagSafe 2 female, J2 ID_LED, J3 2.54mm Output, J4 VCC, J5 GND, Q1 IRF3708

Commit message: Update PCB connect MOSFET tab to output gnd
- Add more labels
- Remove back exposed copper
Connections:
- net GATE: now reaches D1.2 (A), Q1.1 (G), R2.1
Changed lines of the file:
@@
 Wire Wire Line
 	4700 1850 4550 1850
+Text Label 2950 1950 2    50   ~ 0
+GATE
 $EndSCHEMATC
